File: Sensing.kicad_sch (KiCad schematic)
At the start: 0 parts

Commit message: Version 1.1
Other:
- removed sheet ACSense4
- added sheet ACSens4R (ACSens4R.kicad_sch)
Changed lines of the file:
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@@
     (stroke (width 0) (type default))
   )
-  (wire (pts (xy 130.81 148.59) (xy 134.62 148.59))
+  (wire (pts (xy 130.81 147.32) (xy 134.62 147.32))
     (stroke (width 0) (type default))
   )
@@
     (stroke (width 0) (type default))
   )
-  (wire (pts (xy 134.62 161.29) (xy 134.62 158.75))
+  (wire (pts (xy 134.62 161.29) (xy 134.62 157.48))
     (stroke (width 0) (type default))
   )
@@
     (stroke (width 0) (type default))
   )
-  (wire (pts (xy 130.81 153.67) (xy 138.43 153.67))
-    (stroke (width 0) (type default))
-  )
   (wire (pts (xy 91.44 53.34) (xy 105.41 53.34))
     (stroke (width 0) (type default))
@@
     (stroke (width 0) (type default))
   )
-  (wire (pts (xy 134.62 148.59) (xy 134.62 146.05))
+  (wire (pts (xy 134.62 147.32) (xy 134.62 146.05))
+    (stroke (width 0) (type default))
+  )
+  (wire (pts (xy 137.16 82.55) (xy 137.16 78.74))
+    (stroke (width 0) (type default))
+  )
+  (wire (pts (xy 130.81 92.71) (xy 137.16 92.71))
     (stroke (width 0) (type default))
   )
@@
     (stroke (width 0) (type default))
   )
-  (wire (pts (xy 137.16 82.55) (xy 137.16 78.74))
-    (stroke (width 0) (type default))
-  )
-  (wire (pts (xy 130.81 92.71) (xy 137.16 92.71))
-    (stroke (width 0) (type default))
-  )
-  (wire (pts (xy 104.14 156.21) (xy 83.82 156.21))
+  (wire (pts (xy 104.14 154.94) (xy 83.82 154.94))
     (stroke (width 0) (type default))
   )
@@
     (stroke (width 0) (type default))
   )
-  (wire (pts (xy 83.82 156.21) (xy 83.82 121.92))
-    (stroke (width 0) (type default))
-  )
-  (wire (pts (xy 134.62 158.75) (xy 130.81 158.75))
+  (wire (pts (xy 130.81 152.4) (xy 138.43 152.4))
+    (stroke (width 0) (type default))
+  )
+  (wire (pts (xy 83.82 154.94) (xy 83.82 121.92))
+    (stroke (width 0) (type default))
+  )
+  (wire (pts (xy 134.62 157.48) (xy 130.81 157.48))
     (stroke (width 0) (type default))
   )
@@
     (effects (font (size 1.27 1.27)) (justify left))
   )
-  (hierarchical_label "In4" (shape input) (at 138.43 153.67 0) (fields_autoplaced)
+  (hierarchical_label "In4" (shape input) (at 138.43 152.4 0) (fields_autoplaced)
     (effects (font (size 1.27 1.27)) (justify left))
   )
@@
     )
   )
-  (sheet (at 104.14 144.78) (size 26.67 16.51) (fields_autoplaced)
-    (stroke (width 0.1524) (type solid))
-    (fill (color 0 0 0 0.0000))
-    (property "Sheetname" "ACSense4" (at 104.14 144.0684 0)
-      (effects (font (size 1.27 1.27)) (justify left bottom))
-    )
-    (property "Sheetfile" "ACSens.kicad_sch" (at 104.14 161.8746 0)
-      (effects (font (size 1.27 1.27)) (justify left top))
-    )
-    (pin "In~" input (at 104.14 149.86 180)
-      (effects (font (size 1.27 1.27)) (justify left))
-    )
-    (pin "AC{slash}N" input (at 104.14 156.21 180)
-      (effects (font (size 1.27 1.27)) (justify left))
-    )
-    (pin "+Vs" input (at 130.81 148.59 0)
-      (effects (font (size 1.27 1.27)) (justify right))
-    )
-    (pin "Out" input (at 130.81 153.67 0)
-      (effects (font (size 1.27 1.27)) (justify right))
-    )
-    (pin "GND" input (at 130.81 158.75 0)
-      (effects (font (size 1.27 1.27)) (justify right))
-    )
-    (instances
-      (project "WemosD1Mini-8266"
-        (path "/84e8e68d-ec51-4c17-a8b1-603b22d1189f/4578d6cc-30c9-47e3-94c8-3ddc29895f75" (page "5"))
-      )
-    )
-  )
   (sheet (at 104.14 110.49) (size 26.67 16.51) (fields_autoplaced)
     (stroke (width 0.1524) (type solid))
@@
       )
     )
+  )
+  (sheet (at 104.14 144.78) (size 26.67 15.24) (fields_autoplaced)
+    (stroke (width 0.1524) (type solid))
+    (fill (color 0 0 0 0.0000))
+    (property "Sheetname" "ACSens4R" (at 104.14 144.0684 0)
+      (effects (font (size 1.27 1.27)) (justify left bottom))
+    )
+    (property "Sheetfile" "ACSens4R.kicad_sch" (at 104.14 160.6046 0)
+      (effects (font (size 1.27 1.27)) (justify left top))
+    )
+    (pin "In~" input (at 104.14 149.86 180)
+      (effects (font (size 1.27 1.27)) (justify left))
+    )
+    (pin "GND" input (at 130.81 157.48 0)
+      (effects (font (size 1.27 1.27)) (justify right))
+    )
+    (pin "Out" input (at 130.81 152.4 0)
+      (effects (font (size 1.27 1.27)) (justify right))
+    )
+    (pin "+Vs" input (at 130.81 147.32 0)
+      (effects (font (size 1.27 1.27)) (justify right))
+    )
+    (pin "AC{slash}N" input (at 104.14 154.94 180)
+      (effects (font (size 1.27 1.27)) (justify left))
+    )
+    (instances
+      (project "WemosD1Mini-8266"
+        (path "/84e8e68d-ec51-4c17-a8b1-603b22d1189f/4578d6cc-30c9-47e3-94c8-3ddc29895f75" (page "8"))
+      )
+    )
